File: tube-driver_sch-pcb.sch (EAGLE design)
At the start: 114 parts, among them CN1 KS 54, CN2 MINI B USB, CN3 KS 54, CN4 KS 54, CN5 KS 54, CN6 KS 54, CN7 KS 54, CN8 KS 54, CN9 KS 54, Q4 MMBT3904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

Commit message: PWMs routed
Connections:
- removed net USR_BTN_ESP: U5.IO5
- net LED_PWM_0: now also R41.2, U10.EN, U5.IO5; no longer R10.2, U2.EN
- net LED_PWM_1: now also R31.2, U5.IO18, U8.EN; no longer R17.2, U3.EN
- net LED_PWM_2: now also R17.2, U3.EN, U5.IO19; no longer R31.2, U8.EN
- net LED_PWM_3: now also R10.2, U2.EN, U5.IO21; no longer R41.2, U10.EN
Changed lines of the file:
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@@
-</segment>
-</net>
-<net name="USR_BTN_ESP" class="0">
-<segment>
-<pinref part="U5" gate="G$1" pin="IO5"/>
-<wire x1="375.92" y1="111.76" x2="411.48" y2="111.76" width="0.1524" layer="91"/>
-<label x="378.46" y="111.76" size="1.778" layer="95"/>
 </segment>
 </net>
@@
 </segment>
 </net>
+<net name="LED_PWM_0" class="0">
+<segment>
+<pinref part="U5" gate="G$1" pin="IO5"/>
+<wire x1="375.92" y1="111.76" x2="411.48" y2="111.76" width="0.1524" layer="91"/>
+<label x="378.46" y="111.76" size="1.778" layer="95"/>
+</segment>
+</net>
+<net name="LED_PWM_1" class="0">
+<segment>
+<pinref part="U5" gate="G$1" pin="IO18"/>
+<wire x1="375.92" y1="88.9" x2="411.48" y2="88.9" width="0.1524" layer="91"/>
+<label x="378.46" y="88.9" size="1.778" layer="95"/>
+</segment>
+</net>
+<net name="LED_PWM_2" class="0">
+<segment>
+<pinref part="U5" gate="G$1" pin="IO19"/>
+<wire x1="375.92" y1="86.36" x2="411.48" y2="86.36" width="0.1524" layer="91"/>
+<label x="378.46" y="86.36" size="1.778" layer="95"/>
+</segment>
+</net>
+<net name="LED_PWM_3" class="0">
+<segment>
+<pinref part="U5" gate="G$1" pin="IO21"/>
+<wire x1="375.92" y1="81.28" x2="411.48" y2="81.28" width="0.1524" layer="91"/>
+<label x="378.46" y="81.28" size="1.778" layer="95"/>
+</segment>
+</net>
 </nets>
 </sheet>
@@
 </segment>
 </net>
-<net name="LED_PWM_3" class="0">
+<net name="LED_PWM_1" class="0">
+<segment>
+<pinref part="U8" gate="G$1" pin="EN"/>
+<wire x1="58.42" y1="233.68" x2="25.4" y2="233.68" width="0.1524" layer="91"/>
+<pinref part="R31" gate="G$1" pin="2"/>
+<wire x1="25.4" y1="233.68" x2="2.54" y2="233.68" width="0.1524" layer="91"/>
+<wire x1="25.4" y1="218.44" x2="25.4" y2="233.68" width="0.1524" layer="91"/>
+<junction x="25.4" y="233.68"/>
+<label x="5.08" y="233.68" size="1.778" layer="95"/>
+</segment>
+</net>
+<net name="LED_PWM_0" class="0">
 <segment>
 <pinref part="U10" gate="G$1" pin="EN"/>
@@
 <net name="LED_PWM_2" class="0">
 <segment>
-<pinref part="U8" gate="G$1" pin="EN"/>
-<wire x1="58.42" y1="233.68" x2="25.4" y2="233.68" width="0.1524" layer="91"/>
-<pinref part="R31" gate="G$1" pin="2"/>
-<wire x1="25.4" y1="233.68" x2="2.54" y2="233.68" width="0.1524" layer="91"/>
-<wire x1="25.4" y1="218.44" x2="25.4" y2="233.68" width="0.1524" layer="91"/>
-<junction x="25.4" y="233.68"/>
-<label x="5.08" y="233.68" size="1.778" layer="95"/>
-</segment>
-</net>
-<net name="LED_PWM_1" class="0">
-<segment>
 <pinref part="U3" gate="G$1" pin="EN"/>
 <wire x1="58.42" y1="134.62" x2="25.4" y2="134.62" width="0.1524" layer="91"/>
@@
 </segment>
 </net>
-<net name="LED_PWM_0" class="0">
+<net name="LED_PWM_3" class="0">
 <segment>
 <pinref part="U2" gate="G$1" pin="EN"/>
