File: tube-driver_sch-pcb.brd (EAGLE design)
At the start: 100 x 100 mm, 114 parts, among them CN1 KS 54, CN2 MINI B USB, CN3 KS 54, CN4 KS 54, CN5 KS 54, CN6 KS 54, CN7 KS 54, CN8 KS 54, CN9 KS 54, Q4 MMBT3904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

Commit message: Passes DRC
Routing:
- net LED_PWM_2: track 62.4 -> 61.7 mm
Changed lines of the file:
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@@
 <wire x1="46.875" y1="24.375" x2="46.875" y2="25.375" width="0.15" layer="16"/>
 <via x="46.875" y="25.375" extent="1-16" drill="0.3"/>
-<wire x1="78.75" y1="66.36" x2="78" y2="67.11" width="0.15" layer="16"/>
-<wire x1="78" y1="67.11" x2="76.11" y2="67.11" width="0.15" layer="16"/>
+<wire x1="78.75" y1="66.36" x2="75.36" y2="66.36" width="0.15" layer="16"/>
 <wire x1="46.875" y1="37.875" x2="46.875" y2="29.125" width="0.15" layer="16"/>
 <via x="46.875" y="29.125" extent="1-16" drill="0.3"/>
 <wire x1="46.875" y1="29.125" x2="46.875" y2="25.375" width="0.15" layer="1"/>
-<wire x1="76.11" y1="67.11" x2="46.875" y2="37.875" width="0.15" layer="16"/>
+<wire x1="75.36" y1="66.36" x2="46.875" y2="37.875" width="0.15" layer="16"/>
 </signal>
 <signal name="LED_PWM_3">
