File: tl100-4-driver_sch-pcb.brd (EAGLE design)
At the start: 100 x 100 mm, 114 parts, among them CN1 KS 54, CN2 MINI B USB, CN3 KS 54, CN4 KS 54, CN5 KS 54, CN6 KS 54, CN7 KS 54, CN8 KS 54, CN9 KS 54, Q4 MMBT3904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

Commit message: tl100-1 done
Routing:
- net LED_PWM_3: track 82.7 -> 101.1 mm
- net LED_PWM_2: track 61.7 -> 74.8 mm
Changed lines of the file:
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@@
 <contactref element="U6" pad="4"/>
 <contactref element="CN2" pad="D-"/>
-<wire x1="88.225" y1="31.825" x2="88.59289375" y2="31.825" width="0.25" layer="16"/>
 <wire x1="88.225" y1="31.825" x2="88.71789375" y2="31.825" width="0.25" layer="16"/>
 <wire x1="88.71789375" y1="31.825" x2="89.071446875" y2="31.678553125" width="0.25" layer="16" curve="-45"/>
@@
 <wire x1="81.875" y1="16.125" x2="81.875" y2="16.875" width="0.25" layer="16"/>
 <wire x1="80.975" y1="15.225" x2="81.875" y2="16.125" width="0.25" layer="16"/>
-<wire x1="80.375" y1="14.5" x2="80.375" y2="14.625" width="0.25" layer="16"/>
 <wire x1="80.375" y1="14.5" x2="80.975" y2="14.5" width="0.25" layer="16"/>
 <contactref element="D9" pad="K"/>
@@
 <via x="46.875" y="25.375" extent="1-16" drill="0.3"/>
 <wire x1="78.75" y1="66.36" x2="75.36" y2="66.36" width="0.15" layer="16"/>
-<wire x1="46.875" y1="37.875" x2="46.875" y2="29.125" width="0.15" layer="16"/>
+<wire x1="71.5" y1="62.5" x2="71.5" y2="31.375" width="0.15" layer="16"/>
+<wire x1="71.5" y1="31.375" x2="69.375" y2="29.25" width="0.15" layer="16"/>
+<wire x1="69.375" y1="29.25" x2="47" y2="29.25" width="0.15" layer="16"/>
+<wire x1="47" y1="29.25" x2="46.875" y2="29.125" width="0.15" layer="16"/>
 <via x="46.875" y="29.125" extent="1-16" drill="0.3"/>
 <wire x1="46.875" y1="29.125" x2="46.875" y2="25.375" width="0.15" layer="1"/>
-<wire x1="75.36" y1="66.36" x2="46.875" y2="37.875" width="0.15" layer="16"/>
+<wire x1="75.36" y1="66.36" x2="71.5" y2="62.5" width="0.15" layer="16"/>
 </signal>
 <signal name="LED_PWM_3">
@@
 <via x="21.875" y="25.375" extent="1-16" drill="0.3"/>
 <wire x1="78.75" y1="68.9" x2="77.4" y2="68.9" width="0.15" layer="16"/>
-<wire x1="37.625" y1="29.125" x2="21.875" y2="29.125" width="0.15" layer="16"/>
-<via x="21.875" y="29.125" extent="1-16" drill="0.3"/>
-<wire x1="21.875" y1="29.125" x2="21.875" y2="25.375" width="0.15" layer="1"/>
-<wire x1="77.4" y1="68.9" x2="37.625" y2="29.125" width="0.15" layer="16"/>
+<wire x1="69.25" y1="29.625" x2="22" y2="29.625" width="0.15" layer="16"/>
+<via x="22" y="29.625" extent="1-16" drill="0.3"/>
+<wire x1="22" y1="29.625" x2="22" y2="25.5" width="0.15" layer="1"/>
+<wire x1="22" y1="25.5" x2="21.875" y2="25.375" width="0.15" layer="1"/>
+<wire x1="77.4" y1="68.9" x2="72.625" y2="64.125" width="0.15" layer="16"/>
+<wire x1="72.625" y1="64.125" x2="71.125" y2="62.625" width="0.15" layer="16"/>
+<wire x1="71.125" y1="62.625" x2="71.125" y2="31.5" width="0.15" layer="16"/>
+<wire x1="71.125" y1="31.5" x2="69.25" y2="29.625" width="0.15" layer="16"/>
 </signal>
 <signal name="N$5">

Commit message: tl100-4 done
Parts:
- added D10, D11, D12, D8: 36V, DIODES:SOT23-3
- added D13, D14, D15, D16: 1V, DIODES:SC-79
Connections:
- net GND: now also D10.1, D11.1, D12.1, D13.A, D14.A, D15.A, D16.A, D8.1
- net LED0_A: now also D12.2
- net LED0_K: now also D16.K
- net LED1_A: now also D11.2
- net LED1_K: now also D15.K
- net LED2_A: now also D10.2
- net LED2_K: now also D14.K
- net LED3_A: now also D8.2
- net LED3_K: now also D13.K
Routing:
- net ESP32_UART_!RTS: track 24.4 -> 28.3 mm
- net LED2_A: track 99.7 -> 103.1 mm
- net LED1_A: track 99.7 -> 103.1 mm
- net LED0_A: track 99.8 -> 103.2 mm
- net LED1_K: track 32.5 -> 35.0 mm
- net LED0_K: track 32.7 -> 35.2 mm
- net ESP32_EN: track 47.2 -> 49.7 mm
- net GND: track 169.2 -> 166.7 mm, vias 148 -> 155
- net LED_PWM_0: track 65.8 -> 67.2 mm
- net LED2_K: track 30.2 -> 31.6 mm
- net ESP32_UART_RX: track 35.2 -> 36.2 mm
- net LED3_K: track 29.7 -> 30.2 mm
- added copper zone on layer 1, net GND
