File: tl100-4-driver_sch-pcb.sch (EAGLE design)
At the start: 114 parts, among them CN1 KS 54, CN2 MINI B USB, CN3 KS 54, CN4 KS 54, CN5 KS 54, CN6 KS 54, CN7 KS 54, CN8 KS 54, CN9 KS 54, Q4 MMBT3904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

Commit message: tl100-4 done
Parts:
- added D10, D11, D12, D8: 36V, DIODES:GSOT36-HE3-08
- added D13, D14, D15, D16: 1V, DIODES:VESD01C1-02VHG3-08
Connections:
- net GND: now also D10.A, D11.A, D12.A, D13.A, D14.A, D15.A, D16.A, D8.A
- net LED0_A: now also D12.K
- net LED0_K: now also D16.K
- net LED1_A: now also D11.K
- net LED1_K: now also D15.K
- net LED2_A: now also D10.K
- net LED2_K: now also D14.K
- net LED3_A: now also D8.K
- net LED3_K: now also D13.K
Other:
- moved on the sheet: C21, C22, C28, C36, C42, C50, C56, C8
