File: tl100-1v-driver_sch-pcb.brd (EAGLE design)
At the start: 25 x 100 mm, 65 parts, among them CN2 MINI B USB, CN8 KS 54, CN9 KS 54, Q4 MMBT3904, Q5 MMBT3904, U1 CP2102, U10 TPS61500, U11 3.3V BUCK, U4 SN65HVD75D, U5 ESP32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

Commit message: All made to work with seal around the edge
Parts:
- moved C53 3.02 mm to (22.9, 12.1), turned to 90 degrees
- moved C5 2.86 mm to (2.00, 39.4), turned to 90 degrees
- moved C12 2.49 mm to (22.6, 67.6), turned to 90 degrees
- moved R19 1.15 mm to (22.6, 70.4), turned to 90 degrees
- moved R1 1.12 mm to (22.8, 40.5)
- moved C13 1.06 mm to (22.6, 73.1), turned to 90 degrees
- moved C14 1.06 mm to (22.6, 75.9), turned to 270 degrees
Routing:
- net GND: track 85.3 -> 82.5 mm
- net 3V3: track 20.1 -> 18.9 mm
- net ESP32_EN: track 53.0 -> 54.1 mm
- net N$1: track 6.31 -> 5.19 mm
- net N$41: track 1.58 -> 2.21 mm
