File: tl100-4v-driver_sch-pcb.brd (EAGLE design)
At the start: 100 x 100 mm, 122 parts, among them CN1 KS 54, CN2 MINI B USB, CN3 KS 54, CN4 KS 54, CN5 KS 54, CN6 KS 54, CN7 KS 54, CN8 KS 54, CN9 KS 54, Q4 MMBT3904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

Commit message: All made to work with seal around the edge
Parts:
- moved C53 3.02 mm to (97.9, 12.1), turned to 90 degrees
- moved C12 2.49 mm to (97.6, 67.6), turned to 90 degrees
- moved R19 1.15 mm to (97.6, 70.4), turned to 90 degrees
- moved C13 1.06 mm to (97.6, 73.1), turned to 90 degrees
- moved C14 1.06 mm to (97.6, 75.9), turned to 270 degrees
- moved R1 0.75 mm to (98.1, 40.5)
Routing:
- net 3V3: track 20.1 -> 18.9 mm
- net N$1: track 6.31 -> 5.56 mm
- net ESP32_EN: track 49.7 -> 50.3 mm
- net LED_PWM_0: track 67.2 -> 66.6 mm
