File: tl300-4c-driver_sch-pcb.brd (EAGLE design)
At the start: 325 x 325 mm, 122 parts, among them CN1 KS 54, CN2 MINI B USB, CN3 KS 54, CN4 KS 54, CN5 KS 54, CN6 KS 54, CN7 KS 54, CN8 KS 54, CN9 KS 54, Q4 MMBT3904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

Commit message: All made to work with seal around the edge
Parts:
- moved C11 3.02 mm to (12.1, 2.12), turned to 180 degrees
- moved C25 3.02 mm to (2.12, 312.9), turned to 270 degrees
- moved C39 3.02 mm to (312.9, 322.9), turned to 0 degrees
- moved C53 3.02 mm to (322.9, 12.1), turned to 90 degrees
- moved C12 2.49 mm to (322.6, 67.6), turned to 90 degrees
- moved R19 1.15 mm to (322.6, 70.4), turned to 90 degrees
- moved C13 1.06 mm to (322.6, 73.1), turned to 90 degrees
- moved C14 1.06 mm to (322.6, 75.9), turned to 270 degrees
- moved R15 1.06 mm to (3.38, 312.9), turned to 270 degrees
- moved R1 1.00 mm to (322.9, 40.5)
Routing:
- net 3V3: track 20.1 -> 23.0 mm
- net N$1: track 6.31 -> 5.31 mm
- net GND: track 166.7 -> 167.3 mm, vias 162 -> 163
